Commit message: add gazebo simulation

File: chapt6/chapt6_ws/src/robot_description/xacro/tracer/camera.xacro (robot description, xacro)
@@ -4,59 +4,46 @@
         <visual>
             <geometry>
-                <box size="${camera_size_x} ${camera_size_y} ${camera_size_z}"/>
+                <box size="${camera_size_x} ${camera_size_y} ${camera_size_z}" />
             </geometry>
             <material name="camera_color">
-                <color rgba="0.0 0.0 1.0 0.5"/>
+                <color rgba="0.0 0.0 1.0 0.5" />
             </material>
         </visual>
         <collision>
             <geometry>
-                <box size="${camera_size_x} ${camera_size_y} ${camera_size_z}"/>
+                <box size="${camera_size_x} ${camera_size_y} ${camera_size_z}" />
             </geometry>
         </collision>
-        <xacro:box_inertial_matrix m="${camera_mass}" l="${camera_size_x}" w="${camera_size_y}" h="${camera_size_z}"/>
+        <xacro:box_inertial_matrix m="${camera_mass}" l="${camera_size_x}" w="${camera_size_y}"
+            h="${camera_size_z}" />
     </link>
     <joint name="camera2chassis" type="fixed">
-        <parent link="chassis"/>
-        <child link="camera"/>
-        <origin xyz="0.3 0.0 ${chassis_length/2+camera_size_z/2+lidar_length}" rpy="0.0 0.0 0.0"/>
+        <parent link="chassis" />
+        <child link="camera" />
+        <origin xyz="0.3 0.0 ${chassis_length/2+camera_size_z/2+lidar_length}" rpy="0.0 0.0 0.0" />
     </joint>
     <gazebo reference="camera">
-        <!-- 类型设置为 camara -->
-        <sensor type="camera" name="camera_node">
-            <update_rate>20.0</update_rate> <!-- 更新频率 -->
-            <!-- 摄像头基本信息设置 -->
-            <camera name="head">
-                <horizontal_fov>${60.0*pi/180.0}</horizontal_fov>
+        <sensor type="depth" name="camera_sensor">
+            <plugin name="depth_camera" filename="libgazebo_ros_camera.so">
+                <frame_name>camera</frame_name>
+            </plugin>
+            <always_on>true</always_on>
+            <update_rate>10</update_rate>
+            <camera name="camera">
+                <horizontal_fov>1.5009831567</horizontal_fov>
                 <image>
-                    <width>1280</width>
-                    <height>720</height>
+                    <width>800</width>
+                    <height>600</height>
                     <format>R8G8B8</format>
                 </image>
-                <clip>
-                    <near>0.02</near>
-                    <far>300</far>
-                </clip>
-                <noise>
-                    <type>gaussian</type>
-                    <mean>0.0</mean>
-                    <stddev>0.007</stddev>
-                </noise>
+                <distortion>
+                    <k1>0.0</k1>
+                    <k2>0.0</k2>
+                    <k3>0.0</k3>
+                    <p1>0.0</p1>
+                    <p2>0.0</p2>
+                    <center>0.5 0.5</center>
+                </distortion>
             </camera>
-            <!-- 核心插件 -->
-            <plugin name="gazebo_camera" filename="libgazebo_ros_camera.so">
-                <alwaysOn>true</alwaysOn>
-                <updateRate>0.0</updateRate>
-                <cameraName>/camera</cameraName>
-                <imageTopicName>image_raw</imageTopicName>
-                <cameraInfoTopicName>camera_info</cameraInfoTopicName>
-                <frameName>camera</frameName>
-                <hackBaseline>0.07</hackBaseline>
-                <distortionK1>0.0</distortionK1>
-                <distortionK2>0.0</distortionK2>
-                <distortionK3>0.0</distortionK3>
-                <distortionT1>0.0</distortionT1>
-                <distortionT2>0.0</distortionT2>
-            </plugin>
         </sensor>
     </gazebo>

File: chapt6/chapt6_ws/src/robot_description/xacro/tracer/imu.xacro (robot description, xacro)
@@ -4,38 +4,86 @@
         <visual>
             <geometry>
-                <box size="${imu_l} ${imu_w} ${imu_h}"/>
+                <box size="${imu_l} ${imu_w} ${imu_h}" />
             </geometry>
         </visual>
         <collision>
             <geometry>
-                <box size="${imu_l} ${imu_w} ${imu_h}"/>
+                <box size="${imu_l} ${imu_w} ${imu_h}" />
             </geometry>
         </collision>
-        <xacro:box_inertial_matrix m="${imu_m}" l="${imu_l}" w="${imu_w}" h="${imu_h}"/>
+        <xacro:box_inertial_matrix m="${imu_m}" l="${imu_l}" w="${imu_w}" h="${imu_h}" />
     </link>
     <joint name="imu2chassis" type="fixed">
-        <parent link="chassis"/>
-        <child link="imu"/>
-        <origin xyz="0.0 0.0 ${chassis_length/2+imu_h/2}" rpy="0.0 0.0 0.0"/>
+        <parent link="chassis" />
+        <child link="imu" />
+        <origin xyz="0.0 0.0 ${chassis_length/2+imu_h/2}" rpy="0.0 0.0 0.0" />
     </joint>
     <gazebo reference="imu">
-        <material>Gazebo/Orange</material>
-        <gravity>true</gravity>
         <sensor name="imu_sensor" type="imu">
+            <plugin name="imu_plugin" filename="libgazebo_ros_imu_sensor.so">
+                <ros>
+                    <namespace>/</namespace>
+                    <remapping>~/out:=imu</remapping>
+                </ros>
+                <initial_orientation_as_reference>false</initial_orientation_as_reference>
+            </plugin>
+            <update_rate>100</update_rate>
             <always_on>true</always_on>
-            <update_rate>100</update_rate>
-            <visualize>true</visualize>
-            <topic>__default_topic__</topic>
-            <plugin filename="libgazebo_ros_imu_sensor.so" name="imu_plugin">
-                <topicName>imu</topicName>
-                <bodyName>imu</bodyName>
-                <updateRateHZ>100.0</updateRateHZ>
-                <gaussianNoise>0.0</gaussianNoise>
-                <xyzOffset>0 0 0</xyzOffset>
-                <rpyOffset>0 0 0</rpyOffset>
-                <frameName>imu</frameName>
-            </plugin>
-            <pose>0 0 0 0 0 0</pose>
+            <!-- 六轴噪声设置 -->
+            <imu>
+                <angular_velocity>
+                    <x>
+                        <noise type="gaussian">
+                            <mean>0.0</mean>
+                            <stddev>2e-4</stddev>
+                            <bias_mean>0.0000075</bias_mean>
+                            <bias_stddev>0.0000008</bias_stddev>
+                        </noise>
+                    </x>
+                    <y>
+                        <noise type="gaussian">
+                            <mean>0.0</mean>
+                            <stddev>2e-4</stddev>
+                            <bias_mean>0.0000075</bias_mean>
+                            <bias_stddev>0.0000008</bias_stddev>
+                        </noise>
+                    </y>
+                    <z>
+                        <noise type="gaussian">
+                            <mean>0.0</mean>
+                            <stddev>2e-4</stddev>
+                            <bias_mean>0.0000075</bias_mean>
+                            <bias_stddev>0.0000008</bias_stddev>
+                        </noise>
+                    </z>
+                </angular_velocity>
+                <linear_acceleration>
+                    <x>
+                        <noise type="gaussian">
+                            <mean>0.0</mean>
+                            <stddev>1.7e-2</stddev>
+                            <bias_mean>0.1</bias_mean>
+                            <bias_stddev>0.001</bias_stddev>
+                        </noise>
+                    </x>
+                    <y>
+                        <noise type="gaussian">
+                            <mean>0.0</mean>
+                            <stddev>1.7e-2</stddev>
+                            <bias_mean>0.1</bias_mean>
+                            <bias_stddev>0.001</bias_stddev>
+                        </noise>
+                    </y>
+                    <z>
+                        <noise type="gaussian">
+                            <mean>0.0</mean>
+                            <stddev>1.7e-2</stddev>
+                            <bias_mean>0.1</bias_mean>
+                            <bias_stddev>0.001</bias_stddev>
+                        </noise>
+                    </z>
+                </linear_acceleration>
+            </imu>
         </sensor>
-</gazebo>
+    </gazebo>
 </robot>

File: chapt6/chapt6_ws/src/robot_description/xacro/tracer/lidar.xacro (robot description, xacro)
@@ -4,5 +4,5 @@
         <visual>
             <geometry>
-                <cylinder radius="${lidar_radius}" length="${lidar_length}"/>
+                <cylinder radius="${lidar_radius}" length="${lidar_length}" />
             </geometry>
         </visual>
@@ -12,5 +12,5 @@
             </geometry>
         </collision> -->
-        <xacro:cylinder_inertial_matrix m="${lidar_mass}" r="${lidar_radius}" h="${lidar_length}"/>
+        <xacro:cylinder_inertial_matrix m="${lidar_mass}" r="${lidar_radius}" h="${lidar_length}" />
         <transmission name="lidar2chassis_trans">
             <type>transmission_interface/SimpleTransmission</type>
@@ -31,27 +31,40 @@
     </joint> -->
     <joint name="lidar2chassis" type="fixed">
-        <parent link="chassis"/>
-        <child link="lidar"/>
-        <origin xyz="0.0 0.0 ${chassis_length/2+lidar_length/2}" rpy="0.0 0.0 0.0"/>
+        <parent link="chassis" />
+        <child link="lidar" />
+        <origin xyz="0.0 0.0 ${chassis_length/2+lidar_length/2}" rpy="0.0 0.0 0.0" />
     </joint>
     <gazebo reference="lidar">
-        <sensor type="ray" name="rplidar">
+        <sensor name="laserscan" type="ray">
+            <plugin name="laserscan" filename="libgazebo_ros_ray_sensor.so">
+                <ros>
+                    <namespace>/</namespace>
+                    <remapping>~/out:=scan</remapping>
+                </ros>
+                <output_type>sensor_msgs/LaserScan</output_type>
+                <frame_name>lidar</frame_name>
+            </plugin>
+            <always_on>true</always_on>
+            <visualize>true</visualize>
+            <update_rate>5</update_rate>
             <pose>0 0 0 0 0 0</pose>
-            <visualize>true</visualize>
-            <update_rate>20.0</update_rate>
+            <!-- 激光传感器配置 -->
             <ray>
+                <!-- 设置扫描范围 -->
                 <scan>
                     <horizontal>
-                        <samples>720</samples>
-                        <resolution>1</resolution>
-                        <min_angle>-3</min_angle>
-                        <max_angle>3</max_angle>
+                        <samples>360</samples>
+                        <resolution>1.000000</resolution>
+                        <min_angle>0.000000</min_angle>
+                        <max_angle>6.280000</max_angle>
                     </horizontal>
                 </scan>
+                <!-- 设置扫描距离 -->
                 <range>
-                    <min>0.10</min>
-                    <max>30.0</max>
-                    <resolution>0.01</resolution>
+                    <min>0.120000</min>
+                    <max>8.0</max>
+                    <resolution>0.015000</resolution>
                 </range>
+                <!-- 设置噪声 -->
                 <noise>
                     <type>gaussian</type>
@@ -60,8 +73,4 @@
                 </noise>
             </ray>
-            <plugin name="gazebo_rplidar" filename="libgazebo_ros_laser.so">
-                <topicName>/scan</topicName>
-                <frameName>lidar</frameName>
-            </plugin>
         </sensor>
     </gazebo>

File: chapt6/chapt6_ws/src/robot_description/xacro/tracer/spheres.xacro (robot description, xacro)
@@ -24,14 +24,10 @@
             <axis xyz="1 1 1" />
         </joint>
-        <transmission name="${sphere_name}2chassis_trans">
-            <type>transmission_interface/SimpleTransmission</type>
-            <joint name="${sphere_name}2chassis">
-                <hardwareInterface>EffortJointInterface</hardwareInterface>
-            </joint>
-            <actuator name="${sphere_name}2chassis_motor">
-                <mechanicalReduction>1.0</mechanicalReduction>
-                <hardwareInterface>EffortJointInterface</hardwareInterface>
-            </actuator>
-        </transmission>
+        <gaezbo reference = "${sphere_name}_wheel">
+            <mu1 value = "0.0"/>
+            <mu2 value = "0.0"/>
+            <kp value = "1000000000.0"/>
+            <kd value = "1.0"/>
+        </gaezbo>
     </xacro:macro>
     <xacro:sphere_func sphere_name="front" flag = "1"/>

File: chapt6/chapt6_ws/src/robot_description/xacro/tracer/tracer.xacro (robot description, xacro)
@@ -31,8 +31,9 @@
     <xacro:include filename="$(find robot_description)/xacro/tracer/chassis.xacro"/>
     <xacro:include filename="$(find robot_description)/xacro/tracer/lidar.xacro"/>
-    <xacro:include filename="$(find robot_description)/xacro/tracer/camera.xacro"/>
+    <!-- <xacro:include filename="$(find robot_description)/xacro/tracer/camera.xacro"/> -->
     <!-- <xacro:include filename="$(find robot_description)/xacro/tracer/kinect_camera.xacro"/> -->
     <xacro:include filename="$(find robot_description)/xacro/tracer/spheres.xacro"/>
     <xacro:include filename="$(find robot_description)/xacro/tracer/wheels.xacro"/>
-    <xacro:include filename="$(find robot_description)/xacro/tracer/imu.xacro"/>
+    <!-- <xacro:include filename="$(find robot_description)/xacro/robot_ros2_control.xacro"/> -->
+    <!-- <xacro:include filename="$(find robot_description)/xacro/tracer/imu.xacro"/> -->
 </robot>

File: chapt6/chapt6_ws/src/robot_description/xacro/tracer/wheels.xacro (robot description, xacro)
@@ -26,5 +26,5 @@
             <origin xyz="0 ${wheel_dist/2*flag} ${(sphere_radius*2+chassis_length/2-wheel_radius)*-1}" rpy="0 0 0"/>
         </joint>
-        <transmission name="${wheel_name}2chassis_trans">
+        <!-- <transmission name="${wheel_name}2chassis_trans">
             <type>transmission_interface/SimpleTransmission</type>
             <joint name="${wheel_name}2chassis">
@@ -35,5 +35,11 @@
                 <hardwareInterface>hardware_interface/EffortJointInterface</hardwareInterface>
             </actuator>
-        </transmission>
+        </transmission> -->
+        <gaezbo reference = "${wheel_name}_wheel">
+            <mu1 value = "20.0"/>
+            <mu2 value = "20.0"/>
+            <kp value = "1000000000.0"/>
+            <kd value = "1.0"/>
+        </gaezbo>
     </xacro:macro>
     <xacro:wheel_func wheel_name="left" flag = "1"/>
@@ -41,23 +47,19 @@
     <gazebo>
         <plugin name="differential_drive_controller" filename="libgazebo_ros_diff_drive.so">
-            <rosDebugLevel>Debug</rosDebugLevel>
-            <publishWheelTF>false</publishWheelTF>
-            <robotNamespace>/</robotNamespace>
-            <publishTf>1</publishTf>
-            <publishWheelJointState>false</publishWheelJointState>
-            <alwaysOn>true</alwaysOn>
-            <updateRate>100.0</updateRate>
-            <legacyMode>true</legacyMode>
-            <leftJoint>left2chassis</leftJoint> <!-- 左轮 -->
-            <rightJoint>right2chassis</rightJoint> <!-- 右轮 -->
-            <wheelSeparation>${0.6+wheel_length}</wheelSeparation> <!-- 车轮间距 -->
-            <wheelDiameter>${wheel_radius*2}</wheelDiameter> <!-- 车轮直径 -->
-            <broadcastTF>1</broadcastTF>
-            <wheelTorque>30</wheelTorque>
-            <wheelAcceleration>1.8</wheelAcceleration>
-            <commandTopic>/cmd_vel</commandTopic> <!-- 运动控制话题 -->
-            <odometryFrame>/odom</odometryFrame>
-            <odometryTopic>/odom</odometryTopic> <!-- 里程计话题 -->
-            <robotBaseFrame>/base_link</robotBaseFrame> <!-- 根坐标系 -->
+            <ros>
+                <namespace>/</namespace>
+            </ros>
+            <update_rate>30.0</update_rate>
+            <left_joint>left2chassis</left_joint>
+            <right_joint>right2chassis</right_joint>
+            <wheel_separation>${0.6+wheel_length}</wheel_separation>
+            <wheel_diameter>${wheel_radius*2}</wheel_diameter>
+            <max_wheel_torque>20</max_wheel_torque>
+            <max_wheel_acceleration>1.0</max_wheel_acceleration>
+            <publish_odom>true</publish_odom>
+            <publish_odom_tf>true</publish_odom_tf>
+            <publish_wheel_tf>true</publish_wheel_tf>
+            <odometry_frame>odom</odometry_frame>
+            <robot_base_frame>base_link</robot_base_frame>
         </plugin>
     </gazebo>
