Commit message: add autopatrol and README

File: chapt7/chapt7_ws/src/robot_description/xacro/tracer/camera.xacro (robot description, xacro)
@@ -23,8 +23,16 @@
         <origin xyz="0.3 0.0 ${chassis_length/2+camera_size_z/2+lidar_length}" rpy="0.0 0.0 0.0" />
     </joint>
+    <link name="depth_camera_frame"/>
+    <joint name="camera_optical_joint" type="fixed">
+        <parent link="camera"/>
+        <child link="depth_camera_frame"/>
+        <origin
+            xyz="0 0 0"
+            rpy="-1.57079632679 0 -1.57079632679"/>
+    </joint>
     <gazebo reference="camera">
         <sensor type="depth" name="camera_sensor">
             <plugin name="depth_camera" filename="libgazebo_ros_camera.so">
-                <frame_name>camera</frame_name>
+                <frame_name>depth_camera_frame</frame_name>
             </plugin>
             <always_on>true</always_on>

File: chapt7/chapt7_ws/src/robot_description/xacro/tracer/tracer.xacro (robot description, xacro)
@@ -31,5 +31,5 @@
     <xacro:include filename="$(find robot_description)/xacro/tracer/chassis.xacro"/>
     <xacro:include filename="$(find robot_description)/xacro/tracer/lidar.xacro"/>
-    <!-- <xacro:include filename="$(find robot_description)/xacro/tracer/camera.xacro"/> -->
+    <xacro:include filename="$(find robot_description)/xacro/tracer/camera.xacro"/>
     <!-- <xacro:include filename="$(find robot_description)/xacro/tracer/kinect_camera.xacro"/> -->
     <xacro:include filename="$(find robot_description)/xacro/tracer/spheres.xacro"/>
